File: pcb/pmic_dev.kicad_sch (KiCad schematic)
At the start: 56 parts, among them J1 Conn_01x05_Pin, J10 Conn_01x05_Pin, J11 Conn_01x05_Pin, J12 Conn_01x05_Pin, J13 Conn_01x05_Pin, J2 Conn_01x05_Pin, J3 Conn_01x08_Pin, J4 Conn_01x05_Pin, J5 Conn_01x05_Pin, J6 Conn_01x05_Pin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

Commit message: pcb: Update names
Other:
- title: FTDI debug probe -> AVR/PICO/ESP dev board
