File: pcb_esp/esp.kicad_sch (KiCad schematic)
At the start: 13 parts, among them J4 Conn_01x05_Pin, J5 Conn_01x05_Pin, J6 Conn_01x05_Pin, J7 Conn_01x08_Pin, J8 Conn_02x03_Odd_Even, U5 ESP-12F

Commit message: pcb_esp: Version 20240902
Parts:
- R14: renamed from R12; footprint Resistor_SMD:R_0402_1005Metric_Pad0.72x0.64mm_HandSolder -> Resistor_SMD:R_0402_1005Metric
- R15: renamed from R13; footprint Resistor_SMD:R_0402_1005Metric_Pad0.72x0.64mm_HandSolder -> Resistor_SMD:R_0402_1005Metric
- R16: renamed from R14; footprint Resistor_SMD:R_0402_1005Metric_Pad0.72x0.64mm_HandSolder -> Resistor_SMD:R_0402_1005Metric
- R17: renamed from R15; footprint Resistor_SMD:R_0402_1005Metric_Pad0.72x0.64mm_HandSolder -> Resistor_SMD:R_0402_1005Metric
- R18: renamed from R16; footprint Resistor_SMD:R_0402_1005Metric_Pad0.72x0.64mm_HandSolder -> Resistor_SMD:R_0402_1005Metric
- renumbered TP1 to TP2, TP2 to TP3
Connections:
- net GPIO0: now also J8.2 (Pin_2); no longer J8.5 (Pin_5)
- net RST: now also J8.5 (Pin_5); no longer J8.2 (Pin_2)
Changed lines of the file:
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@@
 	)
 	(label "RST"
-		(at 73.66 172.72 0)
-		(fields_autoplaced yes)
-		(effects
-			(font
-				(size 1.27 1.27)
-			)
-			(justify left bottom)
+		(at 60.96 177.8 180)
+		(fields_autoplaced yes)
+		(effects
+			(font
+				(size 1.27 1.27)
+			)
+			(justify right bottom)
 		)
 	)
@@
 	)
 	(label "GPIO0"
-		(at 60.96 177.8 180)
-		(fields_autoplaced yes)
-		(effects
-			(font
-				(size 1.27 1.27)
-			)
-			(justify right bottom)
+		(at 73.66 172.72 0)
+		(fields_autoplaced yes)
+		(effects
+			(font
+				(size 1.27 1.27)
+			)
+			(justify left bottom)
 		)
 	)
@@
 		(dnp no)
 		(fields_autoplaced yes)
-		(property "Reference" "#PWR036"
+		(property "Reference" "#PWR039"
 			(at 78.74 146.05 0)
 			(effects
@@
 			(project "pcb_mini"
 				(path "/fe94bf59-a1f6-472b-a764-daaf1fcf77e5/e37e3070-18fb-4344-a26c-a10679b6218b"
-					(reference "#PWR036")
+					(reference "#PWR039")
 					(unit 1)
 				)
@@
 		(dnp no)
 		(fields_autoplaced yes)
-		(property "Reference" "TP2"
+		(property "Reference" "TP3"
 			(at 93.98 170.6879 0)
 			(effects
@@
 			(project "pcb_mini"
 				(path "/fe94bf59-a1f6-472b-a764-daaf1fcf77e5/e37e3070-18fb-4344-a26c-a10679b6218b"
-					(reference "TP2")
+					(reference "TP3")
 					(unit 1)
 				)
@@
 		(dnp no)
 		(fields_autoplaced yes)
-		(property "Reference" "TP1"
+		(property "Reference" "TP2"
 			(at 93.98 163.0679 0)
 			(effects
@@
 			(project "pcb_mini"
 				(path "/fe94bf59-a1f6-472b-a764-daaf1fcf77e5/e37e3070-18fb-4344-a26c-a10679b6218b"
-					(reference "TP1")
+					(reference "TP2")
 					(unit 1)
 				)
@@
 		(dnp no)
 		(fields_autoplaced yes)
-		(property "Reference" "R15"
+		(property "Reference" "R17"
 			(at 105.41 91.44 90)
 			(effects
@@
 			)
 		)
-		(property "Footprint" "Resistor_SMD:R_0402_1005Metric_Pad0.72x0.64mm_HandSolder"
+		(property "Footprint" "Resistor_SMD:R_0402_1005Metric"
 			(at 102.362 95.25 90)
 			(effects
@@
 			(project "pcb_mini"
 				(path "/fe94bf59-a1f6-472b-a764-daaf1fcf77e5/e37e3070-18fb-4344-a26c-a10679b6218b"
-					(reference "R15")
+					(reference "R17")
 					(unit 1)
 				)
@@
 		(dnp no)
 		(fields_autoplaced yes)
-		(property "Reference" "#PWR039"
+		(property "Reference" "#PWR042"
 			(at 35.56 186.69 0)
 			(effects
@@
 			(project "pcb_mini"
 				(path "/fe94bf59-a1f6-472b-a764-daaf1fcf77e5/e37e3070-18fb-4344-a26c-a10679b6218b"
-					(reference "#PWR039")
+					(reference "#PWR042")
 					(unit 1)
 				)
@@
 		(dnp no)
 		(fields_autoplaced yes)
-		(property "Reference" "#PWR038"
+		(property "Reference" "#PWR041"
 			(at 35.56 161.29 0)
 			(effects
@@
 			(project "pcb_mini"
 				(path "/fe94bf59-a1f6-472b-a764-daaf1fcf77e5/e37e3070-18fb-4344-a26c-a10679b6218b"
-					(reference "#PWR038")
+					(reference "#PWR041")
 					(unit 1)
 				)
@@
 		(dnp no)
 		(fields_autoplaced yes)
-		(property "Reference" "R13"
+		(property "Reference" "R15"
 			(at 59.69 91.44 90)
 			(effects
@@
 			)
 		)
-		(property "Footprint" "Resistor_SMD:R_0402_1005Metric_Pad0.72x0.64mm_HandSolder"
+		(property "Footprint" "Resistor_SMD:R_0402_1005Metric"
 			(at 56.642 95.25 90)
 			(effects
@@
 			(project "pcb_mini"
 				(path "/fe94bf59-a1f6-472b-a764-daaf1fcf77e5/e37e3070-18fb-4344-a26c-a10679b6218b"
-					(reference "R13")
+					(reference "R15")
 					(unit 1)
 				)
@@
 		(dnp no)
 		(fields_autoplaced yes)
-		(property "Reference" "#PWR034"
+		(property "Reference" "#PWR037"
 			(at 104.14 92.71 0)
 			(effects
@@
 			(project "pcb_mini"
 				(path "/fe94bf59-a1f6-472b-a764-daaf1fcf77e5/e37e3070-18fb-4344-a26c-a10679b6218b"
-					(reference "#PWR034")
+					(reference "#PWR037")
 					(unit 1)
 				)
@@
 		(dnp no)
 		(fields_autoplaced yes)
-		(property "Reference" "#PWR035"
+		(property "Reference" "#PWR038"
 			(at 165.1 120.65 0)
 			(effects
@@
 			(project "pcb_mini"
 				(path "/fe94bf59-a1f6-472b-a764-daaf1fcf77e5/e37e3070-18fb-4344-a26c-a10679b6218b"
-					(reference "#PWR035")
+					(reference "#PWR038")
 					(unit 1)
 				)
@@
 		(dnp no)
 		(fields_autoplaced yes)
-		(property "Reference" "#PWR037"
+		(property "Reference" "#PWR040"
 			(at 106.68 146.05 0)
 			(effects
@@
 			(project "pcb_mini"
 				(path "/fe94bf59-a1f6-472b-a764-daaf1fcf77e5/e37e3070-18fb-4344-a26c-a10679b6218b"
-					(reference "#PWR037")
+					(reference "#PWR040")
 					(unit 1)
 				)
@@
 		(dnp no)
 		(fields_autoplaced yes)
-		(property "Reference" "R14"
+		(property "Reference" "R16"
 			(at 100.33 91.44 90)
 			(effects
@@
 			)
 		)
-		(property "Footprint" "Resistor_SMD:R_0402_1005Metric_Pad0.72x0.64mm_HandSolder"
+		(property "Footprint" "Resistor_SMD:R_0402_1005Metric"
 			(at 97.282 95.25 90)
 			(effects
@@
 			(project "pcb_mini"
 				(path "/fe94bf59-a1f6-472b-a764-daaf1fcf77e5/e37e3070-18fb-4344-a26c-a10679b6218b"
-					(reference "R14")
+					(reference "R16")
 					(unit 1)
 				)
@@
 		(dnp no)
 		(fields_autoplaced yes)
-		(property "Reference" "#PWR030"
+		(property "Reference" "#PWR033"
 			(at 53.34 92.71 0)
 			(effects
@@
 			(project "pcb_mini"
 				(path "/fe94bf59-a1f6-472b-a764-daaf1fcf77e5/e37e3070-18fb-4344-a26c-a10679b6218b"
-					(reference "#PWR030")
+					(reference "#PWR033")
 					(unit 1)
 				)
@@
 		(dnp no)
 		(fields_autoplaced yes)
-		(property "Reference" "#PWR040"
+		(property "Reference" "#PWR043"
 			(at 76.2 186.69 0)
 			(effects
@@
 			(project "pcb_mini"
 				(path "/fe94bf59-a1f6-472b-a764-daaf1fcf77e5/e37e3070-18fb-4344-a26c-a10679b6218b"
-					(reference "#PWR040")
+					(reference "#PWR043")
 					(unit 1)
 				)
@@
 		(dnp no)
 		(fields_autoplaced yes)
-		(property "Reference" "#PWR031"
+		(property "Reference" "#PWR034"
 			(at 58.42 92.71 0)
 			(effects
@@
 			(project "pcb_mini"
 				(path "/fe94bf59-a1f6-472b-a764-daaf1fcf77e5/e37e3070-18fb-4344-a26c-a10679b6218b"
-					(reference "#PWR031")
+					(reference "#PWR034")
 					(unit 1)
 				)
@@
 		(dnp no)
 		(fields_autoplaced yes)
-		(property "Reference" "R12"
+		(property "Reference" "R14"
 			(at 54.61 91.44 90)
 			(effects
@@
 			)
 		)
-		(property "Footprint" "Resistor_SMD:R_0402_1005Metric_Pad0.72x0.64mm_HandSolder"
+		(property "Footprint" "Resistor_SMD:R_0402_1005Metric"
 			(at 51.562 95.25 90)
 			(effects
@@
 			(project "pcb_mini"
 				(path "/fe94bf59-a1f6-472b-a764-daaf1fcf77e5/e37e3070-18fb-4344-a26c-a10679b6218b"
-					(reference "R12")
+					(reference "R14")
 					(unit 1)
 				)
@@
 		(dnp no)
 		(fields_autoplaced yes)
-		(property "Reference" "#PWR032"
+		(property "Reference" "#PWR035"
 			(at 78.74 92.71 0)
 			(effects
@@
 			(project "pcb_mini"
 				(path "/fe94bf59-a1f6-472b-a764-daaf1fcf77e5/e37e3070-18fb-4344-a26c-a10679b6218b"
-					(reference "#PWR032")
+					(reference "#PWR035")
 					(unit 1)
 				)
@@
 		(dnp no)
 		(fields_autoplaced yes)
-		(property "Reference" "#PWR029"
+		(property "Reference" "#PWR032"
 			(at 157.48 52.07 0)
 			(effects
@@
 			(project "pcb_mini"
 				(path "/fe94bf59-a1f6-472b-a764-daaf1fcf77e5/e37e3070-18fb-4344-a26c-a10679b6218b"
-					(reference "#PWR029")
+					(reference "#PWR032")
 					(unit 1)
 				)
@@
 		(dnp no)
 		(fields_autoplaced yes)
-		(property "Reference" "R16"
+		(property "Reference" "R18"
 			(at 107.95 129.54 90)
 			(effects
@@
 			)
 		)
-		(property "Footprint" "Resistor_SMD:R_0402_1005Metric_Pad0.72x0.64mm_HandSolder"
+		(property "Footprint" "Resistor_SMD:R_0402_1005Metric"
 			(at 104.902 133.35 90)
 			(effects
@@
 			(project "pcb_mini"
 				(path "/fe94bf59-a1f6-472b-a764-daaf1fcf77e5/e37e3070-18fb-4344-a26c-a10679b6218b"
-					(reference "R16")
+					(reference "R18")
 					(unit 1)
 				)
@@
 		(dnp no)
 		(fields_autoplaced yes)
-		(property "Reference" "#PWR033"
+		(property "Reference" "#PWR036"
 			(at 99.06 92.71 0)
 			(effects
@@
 			(project "pcb_mini"
 				(path "/fe94bf59-a1f6-472b-a764-daaf1fcf77e5/e37e3070-18fb-4344-a26c-a10679b6218b"
-					(reference "#PWR033")
-					(unit 1)
-				)
+					(reference "#PWR036")
+					(unit 1)
+				)
