File: pcb_esp/power.kicad_sch (KiCad schematic)
At the start: 32 parts, among them J1 Conn_01x05_Pin, J2 Conn_01x04_Pin, J3 Conn_02x03_Odd_Even, Q1 DMG2302U, Q2 DMG2301L, SW1 SW_Push, U1 AP2112K-3.3, U2 PCA9306, U3 ATtiny84A-SS, U4 SHT4x

Commit message: pcb_esp: Version 20240902
Parts:
- removed J1: Conn_01x05_Pin, Connector_PinHeader_2.54mm:PinHeader_1x05_P2.54mm_Vertical, symbol Connector:Conn_01x05_Pin
- removed J2: Conn_01x04_Pin, Connector_PinHeader_2.54mm:PinHeader_1x04_P2.54mm_Vertical, symbol Connector:Conn_01x04_Pin
- added C10, C7, C8: 100n, Capacitor_SMD:C_0402_1005Metric, symbol Device:C
- added J1, J2: Conn_01x06, Connector_PinHeader_2.54mm:PinHeader_1x06_P2.54mm_Vertical, symbol Connector_Generic:Conn_01x06
- added Q2, Q4: DMG2301L, Package_TO_SOT_SMD:SOT-23, symbol Transistor_FET:DMG2301L
- added R6, R8: 10k, Resistor_SMD:R_0402_1005Metric, symbol Device:R
- C1, C2, C3, C4, C5, C6: footprint Capacitor_SMD:C_0402_1005Metric_Pad0.74x0.62mm_HandSolder -> Capacitor_SMD:C_0402_1005Metric
- C11: renamed from C8; footprint Capacitor_SMD:C_0402_1005Metric_Pad0.74x0.62mm_HandSolder -> Capacitor_SMD:C_0402_1005Metric
- C9: renamed from C7; footprint Capacitor_SMD:C_0402_1005Metric_Pad0.74x0.62mm_HandSolder -> Capacitor_SMD:C_0402_1005Metric
- LED1: footprint MSL0601RGBU1 -> Library:MSL0601RGBU1
- R1, R2, R3, R4, R5: footprint Resistor_SMD:R_0402_1005Metric_Pad0.72x0.64mm_HandSolder -> Resistor_SMD:R_0402_1005Metric
- R10: renamed from R8; footprint Resistor_SMD:R_0402_1005Metric_Pad0.72x0.64mm_HandSolder -> Resistor_SMD:R_0402_1005Metric
- R11: renamed from R9; footprint Resistor_SMD:R_0402_1005Metric_Pad0.72x0.64mm_HandSolder -> Resistor_SMD:R_0402_1005Metric
- R12: renamed from R10; footprint Resistor_SMD:R_0402_1005Metric_Pad0.72x0.64mm_HandSolder -> Resistor_SMD:R_0402_1005Metric
- R13: renamed from R11; footprint Resistor_SMD:R_0402_1005Metric_Pad0.72x0.64mm_HandSolder -> Resistor_SMD:R_0402_1005Metric
- R7: renamed from R6; footprint Resistor_SMD:R_0402_1005Metric_Pad0.72x0.64mm_HandSolder -> Resistor_SMD:R_0402_1005Metric
- R9: renamed from R7; footprint Resistor_SMD:R_0402_1005Metric_Pad0.72x0.64mm_HandSolder -> Resistor_SMD:R_0402_1005Metric
- renumbered Q2 to Q3
Connections:
- net +3V3: now also Q4.2 (S), R8.1
- net +BATT: now also Q2.2 (S), R6.1
- net GND: now also C10.2, C7.2, C8.2, J1.5 (Pin_5), J1.6 (Pin_6), J2.5 (Pin_5), J2.6 (Pin_6)
- net MOSI: now also J1.3 (Pin_3)
- net PA0: now also C7.1
- net PA4: now also J1.4 (Pin_4)
- net SCL: now also J2.4 (Pin_4)
- net SDA: now also J2.3 (Pin_3)
- net PA1 renamed AUX_EN
- net AUX_EN: now also Q2.1 (G), Q4.1 (G), R6.2, R8.2
- new net AUX_3V3: C10.1, J2.1 (Pin_1), J2.2 (Pin_2), Q4.3 (D)
- new net AUX_VBAT: C8.1, J1.1 (Pin_1), J1.2 (Pin_2), Q2.3 (D)
Other:
- moved on the sheet: C9, Q3, R7
